Commit message: 3/24/26 add rviz and robot body

File: description/robot_core.xacro (robot description, xacro)
@@ -26,30 +26,30 @@
         <parent link="base_link"/>
         <child link="chassis"/>
-        <origin xyz="-0.1 0 0"/>
+        <origin xyz="0 0 0"/>
     </joint>
     <!-- Chassis -->
     <link name="chassis">
         <visual>
-            <origin xyz="0.15 0 0.075"/>
+            <origin xyz="0.125 0 0.0625"/>
             <geometry>
-                <box size="0.3 0.3 0.15"/>
+                <box size="0.25 0.25 0.045"/>
             </geometry>
             <material name="blue"/>
         </visual>
         <collision>
-            <origin xyz="0.15 0 0.075"/>
+            <origin xyz="0.125 0 0.0625"/>
             <geometry>
-                <box size="0.3 0.3 0.15"/>
+                <box size="0.25 0.25 0.045"/>
             </geometry>
         </collision>
-        <xacro:inertial_box mass="0.5" x="0.3" y="0.3" z="0.15">
-            <origin xyz="0.15 0 0.075" rpy="0 0 0"/>
+        <xacro:inertial_box mass="0.5" x="0.25" y="0.25" z="0.045">
+            <origin xyz="0.125 0 0.0625" rpy="0 0 0"/>
         </xacro:inertial_box>
     </link>
-    <!-- Left Wheel  -->
+    <!-- Left Wheel -->
     <joint name="left_wheel_joint" type="continuous">
         <parent link="base_link"/>
         <child link="left_wheel"/>
-        <origin xyz="0 0.175 0" rpy="-${pi/2} 0 0"/>
+        <origin xyz="0.125 0.142 0.0425" rpy="-${pi/2} 0 0"/>
         <axis xyz="0 0 1"/>
     </joint>
@@ -57,5 +57,5 @@
         <visual>
             <geometry>
-                <cylinder radius="0.08" length="0.0334"/>
+                <cylinder radius="0.0425" length="0.0334"/>
             </geometry>
             <material name="black"/>
@@ -63,8 +63,8 @@
         <collision>
             <geometry>
-                <cylinder radius="0.08" length="0.0334"/>
+                <cylinder radius="0.0425" length="0.0334"/>
             </geometry>
         </collision>
-        <xacro:inertial_cylinder mass="0.1" length="0.04" radius="0.08">
+        <xacro:inertial_cylinder mass="0.1" length="0.0334" radius="0.0425">
             <origin xyz="0 0 0" rpy="0 0 0"/>
         </xacro:inertial_cylinder>
@@ -74,5 +74,5 @@
         <parent link="base_link"/>
         <child link="right_wheel"/>
-        <origin xyz="0 -0.175 0" rpy="${pi/2} 0 0"/>
+        <origin xyz="0.125 -0.142 0.0425" rpy="${pi/2} 0 0"/>
         <axis xyz="0 0 1"/>
     </joint>
@@ -80,5 +80,5 @@
         <visual>
             <geometry>
-                <cylinder radius="0.08" length="0.0334"/>
+                <cylinder radius="0.0425" length="0.0334"/>
             </geometry>
             <material name="black"/>
@@ -86,8 +86,8 @@
         <collision>
             <geometry>
-                <cylinder radius="0.08" length="0.0334"/>
+                <cylinder radius="0.0425" length="0.0334"/>
             </geometry>
         </collision>
-        <xacro:inertial_cylinder mass="0.1" length="0.04" radius="0.08">
+        <xacro:inertial_cylinder mass="0.1" length="0.0334" radius="0.0425">
             <origin xyz="0 0 0" rpy="0 0 0"/>
         </xacro:inertial_cylinder>
@@ -95,7 +95,7 @@
     <!-- Caster Wheel 1-->
     <joint name="caster_wheel_1_joint" type="fixed">
-        <parent link="chassis"/>
-        <child link="caster_wheel_1"/>
-        <origin xyz="0.3 0.15 -0.07" rpy="0 0 0"/>
+    <parent link="chassis"/>
+    <child link="caster_wheel_1"/>
+    <origin xyz="0.23 0.1 0.02" rpy="0 0 0"/>
     </joint>
     <link name="caster_wheel_1">
@@ -117,7 +117,7 @@
     <!-- Caster Wheel 2-->
     <joint name="caster_wheel_2_joint" type="fixed">
-        <parent link="chassis"/>
-        <child link="caster_wheel_2"/>
-        <origin xyz="0.3 -0.15 -0.07" rpy="0 0 0"/>
+    <parent link="chassis"/>
+    <child link="caster_wheel_2"/>
+    <origin xyz="0.23 -0.1 0.02" rpy="${pi/2} 0 0"/>
     </joint>
     <link name="caster_wheel_2">
@@ -137,3 +137,47 @@
         </xacro:inertial_sphere>
     </link>
+    <!-- Caster Wheel 3 (Back Left) -->
+<joint name="caster_wheel_3_joint" type="fixed">
+    <parent link="chassis"/>
+    <child link="caster_wheel_3"/>
+    <origin xyz="0.02 0.1 0.02" rpy="0 0 0"/>
+</joint>
+<link name="caster_wheel_3">
+    <visual>
+        <geometry>
+            <sphere radius="0.02"/>
+        </geometry>
+        <material name="black"/>
+    </visual>
+    <collision>
+        <geometry>
+            <sphere radius="0.02"/>
+        </geometry>
+    </collision>
+    <xacro:inertial_sphere mass="0.1" radius="0.02">
+        <origin xyz="0 0 0" rpy="0 0 0"/>
+    </xacro:inertial_sphere>
+</link>
+<!-- Caster Wheel 4 (Back Right) -->
+<joint name="caster_wheel_4_joint" type="fixed">
+    <parent link="chassis"/>
+    <child link="caster_wheel_4"/>
+    <origin xyz="0.02 -0.1 0.02" rpy="${pi/2} 0 0"/>
+</joint>
+<link name="caster_wheel_4">
+    <visual>
+        <geometry>
+            <sphere radius="0.02"/>
+        </geometry>
+        <material name="black"/>
+    </visual>
+    <collision>
+        <geometry>
+            <sphere radius="0.02"/>
+        </geometry>
+    </collision>
+    <xacro:inertial_sphere mass="0.1" radius="0.02">
+        <origin xyz="0 0 0" rpy="0 0 0"/>
+    </xacro:inertial_sphere>
+</link>
 </robot>
