Commit message: work on lidar sim

File: description/lidar.xacro (robot description, xacro)
@@ -4,5 +4,21 @@
         <parent link="chassis"/>
         <child link="laser_frame"/>
-        <origin xyz="0.1 0 0.175" rpy="0 0 0"/>
+        <origin xyz="0.15 0 0.1" rpy="0 0 0"/>
     </joint>
+    <link name="laser_frame">
+        <visual>
+            <geometry>
+                <cylinder radius="0.05" length="0.04"/>
+            </geometry>
+            <material name="orange"/>
+        </visual>
+        <collision>
+            <geometry>
+                <cylinder radius="0.05" length="0.04"/>
+            </geometry>
+        </collision>
+        <xacro:inertial_cylinder mass="0.1" length="0.0334" radius="0.0425">
+            <origin xyz="0.15 0 .1" rpy="0 0 0"/>
+        </xacro:inertial_cylinder>
+    </link>
 </robot>

File: description/robot.urdf.xacro (robot description, xacro)
@@ -3,5 +3,5 @@
     <!-- Example link -->
     <xacro:include filename="robot_core.xacro"/>
-    <!-- <xacro:include filename="lidar.xacro"/> -->
+    <xacro:include filename="lidar.xacro"/>
     <xacro:include filename="gazebo_control.xacro"/>
 </robot>

Commit message: lidar working , glitch in gazebo with 2 robots displaying

File: description/lidar.xacro (robot description, xacro)
@@ -4,10 +4,10 @@
         <parent link="chassis"/>
         <child link="laser_frame"/>
-        <origin xyz="0.1 0 0.175" rpy="0 0 0"/>
+        <origin xyz="0.1 0 0.1045" rpy="0 0 0"/>
     </joint>
     <link name="laser_frame">
         <visual>
             <geometry>
-                <cylinder radius="0.05" length="0.04"/>
+                <cylinder radius="0.01" length="0.01"/>
             </geometry>
             <material name="red"/>
@@ -15,16 +15,14 @@
         <collision>
             <geometry>
-                <cylinder radius="0.05" length="0.04"/>
+                <cylinder radius="0.01" length="0.01"/>
             </geometry>
         </collision>
-        <xacro:inertial_cylinder mass="0.1" length="0.04" radius="0.05">
+        <xacro:inertial_cylinder mass="0.1" length="0.01" radius="0.01">
             <origin xyz="0 0 0" rpy="0 0 0"/>
         </xacro:inertial_cylinder>
     </link>
     <gazebo reference="laser_frame">
-        <sensor name="laser" type="lidar">
+        <sensor name="laser" type="gpu_lidar">
             <topic>scan</topic>
-            <pose>0 0 0 0 0 0</pose>
-            <visualize>false</visualize>
             <update_rate>5</update_rate>
             <lidar>
@@ -43,5 +41,6 @@
                 </range>
             </lidar>
-            <always_on>1</always_on>
+            <gz_frame_id>laser_frame</gz_frame_id>
+            <visualize>false</visualize>
         </sensor>
     </gazebo>

Commit message: lidar irl working

File: description/lidar.xacro (robot description, xacro)
@@ -4,5 +4,5 @@
         <parent link="chassis"/>
         <child link="laser_frame"/>
-        <origin xyz="0.1 0 0.1045" rpy="0 0 0"/>
+        <origin xyz="0.15 0 0.1" rpy="0 0 0"/>
     </joint>
     <link name="laser_frame">
@@ -25,5 +25,5 @@
         <sensor name="laser" type="gpu_lidar">
             <topic>scan</topic>
-            <update_rate>1</update_rate>
+            <update_rate>5</update_rate>
             <lidar>
                 <scan>
