Commit message: working robot with bugs

File: description/camera1.xacro (robot description, xacro)
@@ -4,5 +4,5 @@
         <parent link="chassis"/>
         <child link="camera_link"/>
-        <origin xyz="0.305 0 0.08" rpy="0 0 0"/>
+        <origin xyz="-0.005 0 0.08" rpy="0 0 ${pi}"/>
     </joint>
     <link name="camera_link">

Commit message: rotation fix around center axis

File: description/camera1.xacro (robot description, xacro)
@@ -4,5 +4,5 @@
         <parent link="chassis"/>
         <child link="camera_link"/>
-        <origin xyz="-0.005 0 0.08" rpy="0 0 ${pi}"/>
+        <origin xyz="-0.175 0 0.1" rpy="0 0 ${pi}"/>
     </joint>
     <link name="camera_link">

File: description/lidar.xacro (robot description, xacro)
@@ -4,5 +4,5 @@
         <parent link="chassis"/>
         <child link="laser_frame"/>
-        <origin xyz="0.15 0 0.1" rpy="0 0 0"/>
+        <origin xyz="0.025 0 0.1" rpy="0 0 0"/>
     </joint>
     <link name="laser_frame">

File: description/robot_core.xacro (robot description, xacro)
@@ -31,5 +31,5 @@
     <link name="chassis">
         <visual>
-            <origin xyz="0.125 0 0.0625"/>
+            <origin xyz="0 0 0.0625"/>
             <geometry>
                 <box size="0.25 0.25 0.045"/>
@@ -38,5 +38,5 @@
         </visual>
         <collision>
-            <origin xyz="0.125 0 0.0625"/>
+            <origin xyz="0 0 0.0625"/>
             <geometry>
                 <box size="0.25 0.25 0.045"/>
@@ -44,5 +44,5 @@
         </collision>
         <xacro:inertial_box mass="0.5" x="0.25" y="0.25" z="0.045">
-            <origin xyz="0.125 0 0.0625" rpy="0 0 0"/>
+            <origin xyz="0 0 0.0625" rpy="0 0 0"/>
         </xacro:inertial_box>
     </link>
@@ -51,5 +51,5 @@
         <parent link="base_link"/>
         <child link="left_wheel"/>
-        <origin xyz="0.125 0.142 0.0425" rpy="-${pi/2} 0 0"/>
+        <origin xyz="0 0.142 0.0425" rpy="-${pi/2} 0 0"/>
         <axis xyz="0 0 -1"/>
     </joint>
@@ -74,5 +74,5 @@
         <parent link="base_link"/>
         <child link="right_wheel"/>
-        <origin xyz="0.125 -0.142 0.0425" rpy="${pi/2} 0 0"/>
+        <origin xyz="0 -0.142 0.0425" rpy="${pi/2} 0 0"/>
         <axis xyz="0 0 1"/>
     </joint>
@@ -117,5 +117,5 @@
     <parent link="chassis"/>
     <child link="caster_wheel_1"/>
-    <origin xyz="0.23 0.1 0.02" rpy="0 0 0"/>
+    <origin xyz="0.105 0.1 0.02" rpy="0 0 0"/>
     </joint>
     <link name="caster_wheel_1">
@@ -139,5 +139,5 @@
     <parent link="chassis"/>
     <child link="caster_wheel_2"/>
-    <origin xyz="0.23 -0.1 0.02" rpy="${pi/2} 0 0"/>
+    <origin xyz="0.105 -0.1 0.02" rpy="${pi/2} 0 0"/>
     </joint>
     <link name="caster_wheel_2">
@@ -161,5 +161,5 @@
     <parent link="chassis"/>
     <child link="caster_wheel_3"/>
-    <origin xyz="0.02 0.1 0.02" rpy="0 0 0"/>
+    <origin xyz="-0.105 0.1 0.02" rpy="0 0 0"/>
 </joint>
 <link name="caster_wheel_3">
@@ -183,5 +183,5 @@
     <parent link="chassis"/>
     <child link="caster_wheel_4"/>
-    <origin xyz="0.02 -0.1 0.02" rpy="${pi/2} 0 0"/>
+    <origin xyz="-0.105 -0.1 0.02" rpy="${pi/2} 0 0"/>
 </joint>
 <link name="caster_wheel_4">
