Commit message: major changes with claude for jetson orin nano

File: description/gazebo_control.xacro (robot description, xacro)
@@ -2,19 +2,22 @@
 <robot xmlns:xacro="http://www.ros.org/wiki/xacro">
     <gazebo>
-        <plugin name ="diff_drive" filename="libgazebo_ros_diff_drive.so">
-        <!-- Wheels -->
-        <left_joint>left_wheel_joint</left_joint>
-        <right_joint>right_wheel_joint</right_joint>
-        <wheel_separation>0.184</wheel_separation>
-        <wheel_diameter>0.1</wheel_diameter>
-        <!-- Limits -->
-        <max_wheel_torque>100</max_wheel_torque>
-        <max_wheel_velocity>10</max_wheel_velocity>
-        <!-- output -->
-        <odometry_frame>odom</odometry_frame>
-        <robot_base_frame>base_link</robot_base_frame>
-        <publish_odom>true</publish_odom>
-        <publish_odom_tf>true</publish_odom_tf>
-        <publish_wheel_tf>true</publish_wheel_tf>
+        <plugin filename="ignition-gazebo-diff-drive-system"
+                name="ignition::gazebo::systems::DiffDrive">
+            <!-- Wheels -->
+            <left_joint>left_wheel_joint</left_joint>
+            <right_joint>right_wheel_joint</right_joint>
+            <wheel_separation>0.184</wheel_separation>
+            <wheel_radius>0.0425</wheel_radius>
+            <!-- Limits -->
+            <max_wheel_torque>100</max_wheel_torque>
+            <max_linear_velocity>10</max_linear_velocity>
+            <!-- Topics -->
+            <topic>cmd_vel</topic>
+            <odom_topic>odom</odom_topic>
+            <tf_topic>tf</tf_topic>
+            <!-- Frames -->
+            <frame_id>odom</frame_id>
+            <child_frame_id>base_link</child_frame_id>
+            <odom_publish_frequency>30</odom_publish_frequency>
         </plugin>
     </gazebo>

File: description/lidar.xacro (robot description, xacro)
@@ -1,8 +1,8 @@
 <?xml version="1.0"?>
-<robot xmlns:xacro="http://www.ros.org/wiki/xacro">
+<robot xmlns:xacro="http://www.ros.org/wiki/xacro" >
     <joint name="laser_joint" type="fixed">
         <parent link="chassis"/>
         <child link="laser_frame"/>
-        <origin xyz="0.15 0 0.1" rpy="0 0 0"/>
+        <origin xyz="0.1 0 0.175" rpy="0 0 0"/>
     </joint>
     <link name="laser_frame">
@@ -11,5 +11,5 @@
                 <cylinder radius="0.05" length="0.04"/>
             </geometry>
-            <material name="orange"/>
+            <material name="red"/>
         </visual>
         <collision>
@@ -18,7 +18,31 @@
             </geometry>
         </collision>
-        <xacro:inertial_cylinder mass="0.1" length="0.0334" radius="0.0425">
-            <origin xyz="0.15 0 .1" rpy="0 0 0"/>
+        <xacro:inertial_cylinder mass="0.1" length="0.04" radius="0.05">
+            <origin xyz="0 0 0" rpy="0 0 0"/>
         </xacro:inertial_cylinder>
     </link>
+    <gazebo reference="laser_frame">
+        <sensor name="laser" type="lidar">
+            <topic>scan</topic>
+            <pose>0 0 0 0 0 0</pose>
+            <visualize>false</visualize>
+            <update_rate>5</update_rate>
+            <lidar>
+                <scan>
+                    <horizontal>
+                        <samples>360</samples>
+                        <resolution>1</resolution>
+                        <min_angle>-3.14159</min_angle>
+                        <max_angle>3.14159</max_angle>
+                    </horizontal>
+                </scan>
+                <range>
+                    <min>0.3</min>
+                    <max>12</max>
+                    <resolution>0.01</resolution>
+                </range>
+            </lidar>
+            <always_on>1</always_on>
+        </sensor>
+    </gazebo>
 </robot>

File: description/robot_core.xacro (robot description, xacro)
@@ -47,7 +47,4 @@
         </xacro:inertial_box>
     </link>
-    <gazebo reference="chassis">
-        <material>Gazebo/Blue</material>
-    </gazebo>
     <!-- Left Wheel -->
     <joint name="left_wheel_joint" type="continuous">
@@ -55,5 +52,5 @@
         <child link="left_wheel"/>
         <origin xyz="0.125 0.142 0.0425" rpy="-${pi/2} 0 0"/>
-        <axis xyz="0 0 1"/>
+        <axis xyz="0 0 -1"/>
     </joint>
     <link name="left_wheel">
@@ -73,7 +70,4 @@
         </xacro:inertial_cylinder>
     </link>
-    <gazebo reference="left_wheel">
-        <material>Gazebo/Black</material>
-    </gazebo>
     <!-- Right Wheel -->
     <joint name="right_wheel_joint" type="continuous">
@@ -99,6 +93,23 @@
         </xacro:inertial_cylinder>
     </link>
-    <gazebo reference="right_wheel">
-        <material>Gazebo/Black</material>
+    <gazebo reference="caster_wheel_1">
+        <collision><surface><friction><ode>
+            <mu>0</mu><mu2>0</mu2>
+        </ode></friction></surface></collision>
+    </gazebo>
+    <gazebo reference="caster_wheel_2">
+        <collision><surface><friction><ode>
+            <mu>0</mu><mu2>0</mu2>
+        </ode></friction></surface></collision>
+    </gazebo>
+    <gazebo reference="caster_wheel_3">
+        <collision><surface><friction><ode>
+            <mu>0</mu><mu2>0</mu2>
+        </ode></friction></surface></collision>
+    </gazebo>
+    <gazebo reference="caster_wheel_4">
+        <collision><surface><friction><ode>
+            <mu>0</mu><mu2>0</mu2>
+        </ode></friction></surface></collision>
     </gazebo>
     <!-- Caster Wheel 1-->
@@ -124,7 +135,4 @@
         </xacro:inertial_sphere>
     </link>
-    <gazebo reference="caster_wheel_1">
-        <material>Gazebo/Black</material>
-    </gazebo>
     <!-- Caster Wheel 2-->
     <joint name="caster_wheel_2_joint" type="fixed">
@@ -149,7 +157,4 @@
         </xacro:inertial_sphere>
     </link>
-    <gazebo reference="caster_wheel_2">
-        <material>Gazebo/Black</material>
-    </gazebo>
     <!-- Caster Wheel 3 (Back Left) -->
 <joint name="caster_wheel_3_joint" type="fixed">
@@ -174,7 +179,4 @@
     </xacro:inertial_sphere>
 </link>
-<gazebo reference="caster_wheel_3">
-    <material>Gazebo/Black</material>
-</gazebo>
 <!-- Caster Wheel 4 (Back Right) -->
 <joint name="caster_wheel_4_joint" type="fixed">
@@ -199,6 +201,3 @@
     </xacro:inertial_sphere>
 </link>
-<gazebo reference="caster_wheel_4">
-    <material>Gazebo/Black</material>
-</gazebo>
 </robot>

Commit message: ros2 control extra bits

File: description/gazebo_control.xacro (robot description, xacro)
@@ -5,11 +5,11 @@
                 name="ignition::gazebo::systems::DiffDrive">
             <!-- Wheels -->
-            <left_joint>right_wheel_joint</left_joint>
-            <right_joint>left_wheel_joint</right_joint>
+            <left_joint>left_wheel_joint</left_joint>
+            <right_joint>right_wheel_joint</right_joint>
             <wheel_separation>0.184</wheel_separation>
             <wheel_radius>0.0425</wheel_radius>
             <!-- Limits -->
             <max_wheel_torque>100</max_wheel_torque>
-            <max_linear_velocity>10</max_linear_velocity>
+            <max_linear_velocity>100</max_linear_velocity>
             <!-- Topics -->
             <topic>cmd_vel</topic>

File: description/robot.urdf.xacro (robot description, xacro)
@@ -1,10 +1,13 @@
 <?xml version="1.0"?>
-<robot xmlns:xacro="http://www.ros.org/wiki/xacro"  name="robot">
-    <!-- Example link -->
+<robot xmlns:xacro="http://www.ros.org/wiki/xacro" name="robot">
+    <xacro:arg name="use_ros2_control" default="true"/>
     <xacro:include filename="robot_core.xacro"/>
     <xacro:include filename="lidar.xacro"/>
     <xacro:include filename="camera1.xacro"/>
-    <xacro:include filename="ros2_control.xacro"/>
-    <!-- might need to remove  -->
-    <!-- <xacro:include filename="gazebo_control.xacro"/> -->
+    <xacro:if value="$(arg use_ros2_control)">
+        <xacro:include filename="ros2_control.xacro"/>
+    </xacro:if>
+    <xacro:unless value="$(arg use_ros2_control)">
+        <xacro:include filename="gazebo_control.xacro"/>
+    </xacro:unless>
 </robot>

File: description/robot_core.xacro (robot description, xacro)
@@ -63,5 +63,5 @@
         <collision>
             <geometry>
-                <cylinder radius="0.0425" length="0.0334"/>
+                <sphere radius="0.0425"/>
             </geometry>
         </collision>
@@ -86,5 +86,5 @@
         <collision>
             <geometry>
-                <cylinder radius="0.0425" length="0.0334"/>
+                <sphere radius="0.0425"/>
             </geometry>
         </collision>
