Commit message: updated gazebo

File: description/robot.urdf.xacro (robot description, xacro)
@@ -4,3 +4,4 @@
     <xacro:include filename="robot_core.xacro"/>
     <!-- <xacro:include filename="lidar.xacro"/> -->
+    <xacro:include filename="gazebo_control.xacro"/>
 </robot>

File: description/robot_core.xacro (robot description, xacro)
@@ -47,4 +47,7 @@
         </xacro:inertial_box>
     </link>
+    <gazebo reference="chassis">
+        <material>Gazebo/Blue</material>
+    </gazebo>
     <!-- Left Wheel -->
     <joint name="left_wheel_joint" type="continuous">
@@ -70,4 +73,7 @@
         </xacro:inertial_cylinder>
     </link>
+    <gazebo reference="left_wheel">
+        <material>Gazebo/Black</material>
+    </gazebo>
     <!-- Right Wheel -->
     <joint name="right_wheel_joint" type="continuous">
@@ -93,4 +99,7 @@
         </xacro:inertial_cylinder>
     </link>
+    <gazebo reference="right_wheel">
+        <material>Gazebo/Black</material>
+    </gazebo>
     <!-- Caster Wheel 1-->
     <joint name="caster_wheel_1_joint" type="fixed">
@@ -115,4 +124,7 @@
         </xacro:inertial_sphere>
     </link>
+    <gazebo reference="caster_wheel_1">
+        <material>Gazebo/Black</material>
+    </gazebo>
     <!-- Caster Wheel 2-->
     <joint name="caster_wheel_2_joint" type="fixed">
@@ -137,4 +149,7 @@
         </xacro:inertial_sphere>
     </link>
+    <gazebo reference="caster_wheel_2">
+        <material>Gazebo/Black</material>
+    </gazebo>
     <!-- Caster Wheel 3 (Back Left) -->
 <joint name="caster_wheel_3_joint" type="fixed">
@@ -159,4 +174,7 @@
     </xacro:inertial_sphere>
 </link>
+<gazebo reference="caster_wheel_3">
+    <material>Gazebo/Black</material>
+</gazebo>
 <!-- Caster Wheel 4 (Back Right) -->
 <joint name="caster_wheel_4_joint" type="fixed">
@@ -181,3 +199,6 @@
     </xacro:inertial_sphere>
 </link>
+<gazebo reference="caster_wheel_4">
+    <material>Gazebo/Black</material>
+</gazebo>
 </robot>

Commit message: live robot with controller

File: description/robot.urdf.xacro (robot description, xacro)
@@ -1,4 +1,15 @@
 <?xml version="1.0"?>
 <robot xmlns:xacro="http://www.ros.org/wiki/xacro" name="robot">
+    <!--
+    CONTROL MODE SWITCH
+    ═══════════════════
+    use_ros2_control:=true  → real robot (diffdrive_arduino Arduino hardware plugin)
+                              uses: ros2_control.xacro
+                              launch: launch_robot.launch2.py
+    use_ros2_control:=false → simulation (Ignition Gazebo native DiffDrive plugin)
+                              uses: gazebo_control.xacro
+                              launch: launch_sim.launch.py
+    This argument is set automatically by the launch files — you do not need to set it manually.
+    -->
     <xacro:arg name="use_ros2_control" default="true"/>
     <xacro:include filename="robot_core.xacro"/>

File: description/ros2_control.xacro (robot description, xacro)
@@ -1,4 +1,37 @@
 <?xml version="1.0"?>
 <robot xmlns:xacro="http://www.ros.org/wiki/xacro">
+    <ros2_control name="RealRobot" type="system">
+        <hardware>
+            <!-- DiffDriveArduino: open-loop PWM, no encoder feedback
+                 Sends: o leftPWM rightPWM (-255 to 255) over serial
+                 max_motor_speed_rads: tune to your motors (rad/s at full PWM) -->
+            <plugin>diffdrive_arduino/DiffDriveArduino</plugin>
+            <param name="left_wheel_name">left_wheel_joint</param>
+            <param name="right_wheel_name">right_wheel_joint</param>
+            <param name="loop_rate">30</param>
+            <param name="device">/dev/ttyACM0</param>
+            <param name="baud_rate">57600</param>
+            <param name="timeout">1000</param>
+            <param name="enc_counts_per_rev">3450</param>
+            <param name="max_motor_speed_rads">5.0</param>
+        </hardware>
+        <joint name="left_wheel_joint">
+            <command_interface name="velocity">
+                <param name="min">-10</param>
+                <param name="max">10</param>
+            </command_interface>
+            <state_interface name="velocity"/>
+            <state_interface name="position"/>
+        </joint>
+        <joint name="right_wheel_joint">
+            <command_interface name="velocity">
+                <param name="min">-10</param>
+                <param name="max">10</param>
+            </command_interface>
+            <state_interface name="velocity"/>
+            <state_interface name="position"/>
+        </joint>
+    </ros2_control>
+    <!--
     <ros2_control name="GazeboSystem" type="system">
         <hardware>
@@ -22,9 +55,4 @@
         </joint>
     </ros2_control>
-    <gazebo>
-        <plugin filename="gz_ros2_control-system"
-                name="gz_ros2_control::GazeboSimROS2ControlPlugin">
-            <parameters>$(find my_bot)/config/my_controller.yaml</parameters>
-        </plugin>
-    </gazebo>
+    -->
 </robot>
